File: 0000.010B.kicad_sch (KiCad schematic)
At the start: 42 parts, among them J5 M3, J6 M3, J7 M3, Q1 50N10, Q2 50N10, U1 IRS2184, U4 INA280A1xDCK

Commit message: Changed MCU to AT90PWM316-16M - much higher PWM frequency than the Atiny. Smaller inductor and replaced electrolytic capacitors with ceramic.
Parts:
- removed C10, C15, C16, C17, C8, C9: 100, Capacitor_SMD:CP_Elec_10x10, symbol Device:C_Polarized
- removed U1: IRS2184, Package_SO:SOIC-8_3.9x4.9mm_P1.27mm, symbol Driver_FET:IRS2184
- added C10, C15, C16, C17, C3, C6, C8, C9: 156, Capacitor_SMD:C_2220_5750Metric, symbol Device:C
- added U6: IRS2181, Package_SO:SOIC-8_3.9x4.9mm_P1.27mm, symbol Driver_FET:IRS2181
- L1: footprint HR_parts:L_TOROID_D30_2P_H_2 -> Inductor_SMD:L_Vishay_IHLP-6767
Connections:
- net +12V: now also U6.5 (VCC)
- net +PV: now also C10.1, C17.1, C8.1, C9.1
- net GND: now also C10.2, C15.2, C16.2, C17.2, C3.2, C6.2, C8.2, C9.2, U6.3 (COM)
- net VBUS: now also C15.1, C16.1, C3.1, C6.1
- net at D3.1 (K), R23.1, R7.2: now also U6.7 (HO)
- net at C4.2, L1.1, Q1.2 (S)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: now also U6.6 (VS)
- net at D4.1 (K), R24.1, R9.2: now also U6.4 (LO)
- net at C4.1: now also U6.8 (VB)
- new net PWMH: U6.1 (HIN)
- new net PWML: U6.2 (LIN)
Other:
- sheet Controller ports: added PWMH, PWML; removed PWM, SWEN
- moved on the sheet: C31, C32, F4, J5, J6, L3, L4, NT1, NT2, R1
