File: local_psu.kicad_sch (KiCad schematic)
At the start: 21 parts, among them U3 LMR71915, U5 L78L05_SOT89

Commit message: Temperature sensor added as the AT90PWM316 does not have an internal one.
Parts:
- added C36: 104, Capacitor_SMD:C_0805_2012Metric, symbol Device:C
Connections:
- net +5V: now also C36.1
- net GND: now also C36.2
Changed lines of the file:
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@@
+	)
+	(junction
+		(at 226.06 69.85)
+		(diameter 0)
+		(color 0 0 0 0)
 	)
 	(junction
@@
 	(wire
 		(pts
+			(xy 232.41 59.69) (xy 232.41 60.96)
+		)
+		(stroke
+			(width 0)
+			(type default)
+		)
+	)
+	(wire
+		(pts
 			(xy 207.01 69.85) (xy 213.36 69.85)
 		)
@@
 	(wire
 		(pts
+			(xy 226.06 59.69) (xy 232.41 59.69)
+		)
+		(stroke
+			(width 0)
+			(type default)
+		)
+	)
+	(wire
+		(pts
 			(xy 138.43 69.85) (xy 138.43 68.58)
 		)
@@
 	(wire
 		(pts
+			(xy 232.41 68.58) (xy 232.41 69.85)
+		)
+		(stroke
+			(width 0)
+			(type default)
+		)
+	)
+	(wire
+		(pts
 			(xy 213.36 59.69) (xy 213.36 60.96)
 		)
@@
 		(pts
 			(xy 158.75 57.15) (xy 158.75 59.69)
+		)
+		(stroke
+			(width 0)
+			(type default)
+		)
+	)
+	(wire
+		(pts
+			(xy 226.06 69.85) (xy 232.41 69.85)
 		)
 		(stroke
@@
 					(unit 1)
 				)
+			)
+		)
+	)
+	(symbol
+		(lib_id "Device:C")
+		(at 232.41 64.77 0)
+		(unit 1)
+		(body_style 1)
+		(exclude_from_sim no)
+		(in_bom yes)
+		(on_board yes)
+		(in_pos_files yes)
+		(dnp no)
+		(property "Reference" "C36"
+			(at 233.68 62.23 0)
+			(show_name no)
+			(do_not_autoplace no)
+			(effects
+				(font
+					(size 1.27 1.27)
+				)
+				(justify left)
+			)
+		)
+		(property "Value" "104"
+			(at 233.68 67.31 0)
+			(show_name no)
+			(do_not_autoplace no)
+			(effects
+				(font
+					(size 1.27 1.27)
+				)
+				(justify left)
+			)
+		)
+		(property "Footprint" "Capacitor_SMD:C_0805_2012Metric"
+			(at 233.3752 68.58 0)
+			(hide yes)
+			(show_name no)
+			(do_not_autoplace no)
+			(effects
+				(font
+					(size 1.27 1.27)
+				)
+			)
+		)
+		(property "Datasheet" ""
+			(at 232.41 64.77 0)
+			(hide yes)
+			(show_name no)
+			(do_not_autoplace no)
+			(effects
+				(font
+					(size 1.27 1.27)
+				)
+			)
+		)
+		(property "Description" "Unpolarized capacitor"
+			(at 232.41 64.77 0)
+			(hide yes)
+			(show_name no)
+			(do_not_autoplace no)
+			(effects
+				(font
+					(size 1.27 1.27)
+				)
+			)
+		)
+		(pin "2"
+		)
+		(pin "1"
+		)
+		(instances
+			(project "0000.010B"
+				(path "/7b1b7ec5-60f7-444b-a8f9-887f2618112b/30bc3af1-3fcd-40b8-b7cf-f89c2aa37bc5"
+					(reference "C36")
+					(unit 1)
+				)

Commit message: Missing component values added.
Parts:
- C5: value 103 -> 102
- L2: value 10 -> 33
- R11: value R -> 100K
- R2: value R -> 1M
- R3: value R -> 62K
- R4: value R -> 68K
- R5: value R -> 24K
- R6: value R -> 2K
Changed lines of the file:
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@@
 			)
 		)
-		(property "Value" "103"
+		(property "Value" "102"
 			(at 157.48 77.47 0)
 			(show_name no)
@@
 			)
 		)
-		(property "Value" "R"
+		(property "Value" "68K"
 			(at 120.65 88.9 90)
 			(show_name no)
@@
 			)
 		)
-		(property "Value" "R"
+		(property "Value" "2K"
 			(at 165.1 85.09 90)
 			(show_name no)
@@
 			)
 		)
-		(property "Value" "R"
+		(property "Value" "62K"
 			(at 113.03 74.93 90)
 			(show_name no)
@@
 			)
 		)
-		(property "Value" "R"
+		(property "Value" "24K"
 			(at 165.1 64.77 90)
 			(show_name no)
@@
 			)
 		)
-		(property "Value" "10"
+		(property "Value" "33"
 			(at 151.13 60.96 90)
 			(show_name no)
@@
 			)
 		)
-		(property "Value" "R"
+		(property "Value" "1M"
 			(at 113.03 64.77 90)
 			(show_name no)
@@
 			)
 		)
-		(property "Value" "R"
+		(property "Value" "100K"
 			(at 146.05 64.77 90)
 			(show_name no)
